File: kicad/configuration.kicad_sch (KiCad schematic)
At the start: 34 parts, among them J4 USB C, J5 HIC SWD, U2 MIMXRT1171DVMAB, U7 W25Q64JWUUIQ, U8 MKL26Z128VFM4, Y2 16MHz

Commit message: added remaining footprints
Parts:
- C39: footprint (none) -> Capacitor_SMD:C_0201_0603Metric
- FB1: footprint (none) -> Inductor_SMD:L_0402_1005Metric
- R9: footprint (none) -> Resistor_SMD:R_0201_0603Metric
- U8: footprint Package_DFN_QFN:QFN-32-1EP_5x5mm_P0.5mm_EP3.45x3.45mm -> project_footprints:MKL26Z128VFM4
Other:
- note added: "TODO: ESD diodes?"
Changed lines of the file:
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@@
 		(comment 2 "© 2026, Theta Machines LLC.")
 	)
+	(text "TODO: ESD diodes?"
+		(exclude_from_sim no)
+		(at 82.296 135.636 0)
+		(effects
+			(font
+				(size 1.27 1.27)
+			)
+		)
+	)
 	(junction
 		(at 78.74 127)
@@
 			)
 		)
-		(property "Footprint" "Package_DFN_QFN:QFN-32-1EP_5x5mm_P0.5mm_EP3.45x3.45mm"
+		(property "Footprint" "project_footprints:MKL26Z128VFM4"
 			(at 48.26 114.554 0)
 			(hide yes)
@@
 			)
 		)
-		(property "Footprint" ""
+		(property "Footprint" "Capacitor_SMD:C_0201_0603Metric"
 			(at 110.49 162.56 0)
 			(hide yes)
@@
 			)
 		)
-		(property "Footprint" ""
+		(property "Footprint" "Inductor_SMD:L_0402_1005Metric"
 			(at 81.28 109.982 90)
 			(hide yes)
@@
 			)
 		)
-		(property "Footprint" ""
+		(property "Footprint" "Resistor_SMD:R_0201_0603Metric"
 			(at 96.52 110.49 0)
 			(hide yes)

Commit message: removed USB host and 1.8V DAC
Parts:
- renumbered C31 to C29, C32 to C30, C33 to C31, C34 to C32, C35 to C33, C36 to C34, C37 to C35, C38 to C36, C39 to C37, J4 to J3, J5 to J4, U2 to U1, U7 to U6, U8 to U7
Other:
- note removed: "TODO: ESD diodes?"

Commit message: finished preliminary routing
Parts:
- U7: footprint project_footprints:MKL26Z128VFM4 -> Package_DFN_QFN:QFN-32-1EP_5x5mm_P0.5mm_EP3.45x3.45mm
Connections:
- net at R24.2, U1.P6 (GPIO_LPSR_02): now also U7.32 (PTD7); no longer U7.???
- net at R22.1, U1.T7 (GPIO_LPSR_03): now also U7.1 (PTE0); no longer U7.???
Changed lines of the file:
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@@
 		(in_pos_files yes)
 		(dnp no)
-		(property "Reference" "#PWR047"
+		(property "Reference" "#PWR052"
 			(at 90.17 127 0)
 			(hide yes)
@@
 			(project "DEV-G2-NANO"
 				(path "/b6656e4d-fdee-4b90-a905-7068c060191f/45e1da5b-d52f-4e94-b563-4995febadb51"
-					(reference "#PWR047")
+					(reference "#PWR052")
 					(unit 1)
 				)
@@
 		(in_pos_files yes)
 		(dnp no)
-		(property "Reference" "#PWR056"
+		(property "Reference" "#PWR061"
 			(at 110.49 171.45 0)
 			(hide yes)
@@
 			(project "DEV-G2-NANO"
 				(path "/b6656e4d-fdee-4b90-a905-7068c060191f/45e1da5b-d52f-4e94-b563-4995febadb51"
-					(reference "#PWR056")
+					(reference "#PWR061")
 					(unit 1)
 				)
@@
 		(in_pos_files yes)
 		(dnp no)
-		(property "Reference" "#PWR044"
+		(property "Reference" "#PWR049"
 			(at 96.52 109.22 0)
 			(hide yes)
@@
 			(project "DEV-G2-NANO"
 				(path "/b6656e4d-fdee-4b90-a905-7068c060191f/45e1da5b-d52f-4e94-b563-4995febadb51"
-					(reference "#PWR044")
+					(reference "#PWR049")
 					(unit 1)
 				)
@@
 		(in_pos_files yes)
 		(dnp no)
-		(property "Reference" "#PWR057"
+		(property "Reference" "#PWR062"
 			(at 134.62 176.53 0)
 			(hide yes)
@@
 			(project "DEV-G2-NANO"
 				(path "/b6656e4d-fdee-4b90-a905-7068c060191f/45e1da5b-d52f-4e94-b563-4995febadb51"
-					(reference "#PWR057")
+					(reference "#PWR062")
 					(unit 1)
 				)
@@
 		(in_pos_files yes)
 		(dnp no)
-		(property "Reference" "#PWR049"
+		(property "Reference" "#PWR054"
 			(at 194.31 134.62 0)
 			(hide yes)
@@
 			(project "DEV-G2-NANO"
 				(path "/b6656e4d-fdee-4b90-a905-7068c060191f/45e1da5b-d52f-4e94-b563-4995febadb51"
-					(reference "#PWR049")
+					(reference "#PWR054")
 					(unit 1)
 				)
@@
 		(in_pos_files yes)
 		(dnp no)
-		(property "Reference" "#PWR040"
+		(property "Reference" "#PWR045"
 			(at 151.13 95.25 0)
 			(hide yes)
@@
 			(project "DEV-G2-NANO"
 				(path "/b6656e4d-fdee-4b90-a905-7068c060191f/45e1da5b-d52f-4e94-b563-4995febadb51"
-					(reference "#PWR040")
+					(reference "#PWR045")
 					(unit 1)
 				)
@@
 		(in_pos_files yes)
 		(dnp no)
-		(property "Reference" "#PWR041"
+		(property "Reference" "#PWR046"
 			(at 194.31 101.6 0)
 			(hide yes)
@@
 			(project "DEV-G2-NANO"
 				(path "/b6656e4d-fdee-4b90-a905-7068c060191f/45e1da5b-d52f-4e94-b563-4995febadb51"
-					(reference "#PWR041")
+					(reference "#PWR046")
 					(unit 1)
 				)
@@
 		(in_pos_files yes)
 		(dnp no)
-		(property "Reference" "#PWR054"
+		(property "Reference" "#PWR059"
 			(at 92.71 161.29 0)
 			(hide yes)
@@
 			(project "DEV-G2-NANO"
 				(path "/b6656e4d-fdee-4b90-a905-7068c060191f/45e1da5b-d52f-4e94-b563-4995febadb51"
-					(reference "#PWR054")
+					(reference "#PWR059")
 					(unit 1)
 				)
@@
 		(in_pos_files yes)
 		(dnp no)
-		(property "Reference" "#PWR052"
+		(property "Reference" "#PWR057"
 			(at 299.72 144.78 0)
 			(hide yes)
@@
 			(project "DEV-G2-NANO"
 				(path "/b6656e4d-fdee-4b90-a905-7068c060191f/45e1da5b-d52f-4e94-b563-4995febadb51"
-					(reference "#PWR052")
+					(reference "#PWR057")
 					(unit 1)
 				)
@@
 			)
 		)
-		(property "Footprint" "project_footprints:MKL26Z128VFM4"
+		(property "Footprint" "Package_DFN_QFN:QFN-32-1EP_5x5mm_P0.5mm_EP3.45x3.45mm"
 			(at 48.26 114.554 0)
 			(hide yes)
@@
 		(pin "31"
 		)
-		(pin "???"
-		)
-		(pin "???"
-		)
 		(instances
 			(project "DEV-G2-NANO"
@@
 		(in_pos_files yes)
 		(dnp no)
-		(property "Reference" "#PWR045"
+		(property "Reference" "#PWR050"
 			(at 130.81 120.65 0)
 			(hide yes)
@@
 			(project "DEV-G2-NANO"
 				(path "/b6656e4d-fdee-4b90-a905-7068c060191f/45e1da5b-d52f-4e94-b563-4995febadb51"
-					(reference "#PWR045")
+					(reference "#PWR050")
 					(unit 1)
 				)
@@
 		(in_pos_files yes)
 		(dnp no)
-		(property "Reference" "#PWR051"
+		(property "Reference" "#PWR056"
 			(at 313.69 140.97 0)
 			(hide yes)
@@
 			(project "DEV-G2-NANO"
 				(path "/b6656e4d-fdee-4b90-a905-7068c060191f/45e1da5b-d52f-4e94-b563-4995febadb51"
-					(reference "#PWR051")
+					(reference "#PWR056")
 					(unit 1)
 				)
@@
 		(in_pos_files yes)
 		(dnp no)
-		(property "Reference" "#PWR048"
+		(property "Reference" "#PWR053"
 			(at 96.52 127 0)
 			(hide yes)
@@
 			(project "DEV-G2-NANO"
 				(path "/b6656e4d-fdee-4b90-a905-7068c060191f/45e1da5b-d52f-4e94-b563-4995febadb51"
-					(reference "#PWR048")
+					(reference "#PWR053")
 					(unit 1)
 				)
@@
 		(in_pos_files yes)
 		(dnp no)
-		(property "Reference" "#PWR053"
+		(property "Reference" "#PWR058"
 			(at 59.69 161.29 0)
 			(hide yes)
@@
 			(project "DEV-G2-NANO"
 				(path "/b6656e4d-fdee-4b90-a905-7068c060191f/45e1da5b-d52f-4e94-b563-4995febadb51"
-					(reference "#PWR053")
+					(reference "#PWR058")
 					(unit 1)
 				)
@@
 		(in_pos_files yes)
 		(dnp no)
-		(property "Reference" "#PWR043"
+		(property "Reference" "#PWR048"
 			(at 151.13 107.95 0)
 			(hide yes)
@@
 			(project "DEV-G2-NANO"
 				(path "/b6656e4d-fdee-4b90-a905-7068c060191f/45e1da5b-d52f-4e94-b563-4995febadb51"
-					(reference "#PWR043")
+					(reference "#PWR048")
 					(unit 1)
 				)
@@
 		(in_pos_files yes)
 		(dnp no)
-		(property "Reference" "#PWR042"
+		(property "Reference" "#PWR047"
 			(at 120.65 107.95 0)
 			(hide yes)
@@
 			(project "DEV-G2-NANO"
 				(path "/b6656e4d-fdee-4b90-a905-7068c060191f/45e1da5b-d52f-4e94-b563-4995febadb51"
-					(reference "#PWR042")
+					(reference "#PWR047")
 					(unit 1)
 				)
@@
 		(in_pos_files yes)
 		(dnp no)
-		(property "Reference" "#PWR055"
+		(property "Reference" "#PWR060"
 			(at 161.29 163.83 0)
 			(hide yes)
@@
 			(project "DEV-G2-NANO"
 				(path "/b6656e4d-fdee-4b90-a905-7068c060191f/45e1da5b-d52f-4e94-b563-4995febadb51"
-					(reference "#PWR055")
+					(reference "#PWR060")
 					(unit 1)
 				)
@@
 		(in_pos_files yes)
 		(dnp no)
-		(property "Reference" "#PWR050"
+		(property "Reference" "#PWR055"
 			(at 161.29 133.35 0)
 			(hide yes)
@@
 			(project "DEV-G2-NANO"
 				(path "/b6656e4d-fdee-4b90-a905-7068c060191f/45e1da5b-d52f-4e94-b563-4995febadb51"
-					(reference "#PWR050")
+					(reference "#PWR055")
 					(unit 1)
 				)
@@
 		(in_pos_files yes)
 		(dnp no)
-		(property "Reference" "#PWR046"
+		(property "Reference" "#PWR051"
 			(at 137.16 120.65 0)
 			(hide yes)
@@
 			(project "DEV-G2-NANO"
 				(path "/b6656e4d-fdee-4b90-a905-7068c060191f/45e1da5b-d52f-4e94-b563-4995febadb51"
-					(reference "#PWR046")
+					(reference "#PWR051")
 					(unit 1)
 				)
@@
 		(in_pos_files yes)
 		(dnp no)
-		(property "Reference" "#PWR039"
+		(property "Reference" "#PWR044"
 			(at 120.65 95.25 0)
 			(hide yes)
@@
 			(project "DEV-G2-NANO"
 				(path "/b6656e4d-fdee-4b90-a905-7068c060191f/45e1da5b-d52f-4e94-b563-4995febadb51"
-					(reference "#PWR039")
+					(reference "#PWR044")
 					(unit 1)
 				)

Commit message: added stitching vias and made cosmetic changes
Parts:
- U7: footprint Package_DFN_QFN:QFN-32-1EP_5x5mm_P0.5mm_EP3.45x3.45mm -> project_footprints:MKL26Z128VFM4
Changed lines of the file:
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@@
 			)
 		)
-		(property "Footprint" "Package_DFN_QFN:QFN-32-1EP_5x5mm_P0.5mm_EP3.45x3.45mm"
+		(property "Footprint" "project_footprints:MKL26Z128VFM4"
 			(at 48.26 114.554 0)
 			(hide yes)
